Commit message: robot

File: urdf/urdf/robot_model.urdf (robot description, URDF)
Before this commit: robot Staubli, 7 links, 6 joints
Joints:
- removed joint BaseToLink_1
- removed joint Link_1ToLink_2
- removed joint Link_2ToLink_3
- removed joint Link_3ToLink_4
- removed joint Link_4ToLink_5
- removed joint Link_5ToLink_6
- added joint Joint_1: type continuous, parent base_link, child link_1, origin xyz=0 0 0.375 rpy=-1.57 0 0, axis 0 1 0, limit lower=-2.96 upper=2.96 effort=300 velocity=1
- added joint Joint_2: type continuous, parent link_1, child link_2, origin xyz=0.0 0.0 0.0 rpy=0 0 0, axis 0 0 1, limit lower=-2.96 upper=2.96 effort=300 velocity=1
- added joint Joint_3: type continuous, parent link_2, child link_3, origin xyz=0 -0.4 0.02 rpy=0 0 0, axis 0 0 1, limit lower=-2.96 upper=2.96 effort=300 velocity=1
- added joint Joint_4: type continuous, parent link_3, child link_4, origin xyz=0 0 0 rpy=1.57 0 0, axis 0 0 1
- added joint Joint_5: type continuous, parent link_4, child link_5, origin xyz=0 0 0.45 rpy=-1.57 0 0, axis 0 0 1, limit lower=-2.96 upper=2.96 effort=300 velocity=1
- added joint Joint_6: type continuous, parent link_5, child link_6, origin xyz=0 -0.07 0 rpy=1.57 0 0, axis 0 0 1, limit lower=-2.96 upper=2.96 effort=300 velocity=1

Commit message: robot

File: urdf/urdf/robot_model.urdf (robot description, URDF)
Before this commit: robot Staubli, 7 links, 6 joints
Joints:
- joint Joint_1: type continuous -> continuous 

Commit message: robot

File: urdf/urdf/robot_model.urdf (robot description, URDF)
Before this commit: robot Staubli, 7 links, 6 joints
Joints:
- joint Joint_1: type continuous  -> continuous

Commit message: 1.57 -> 1.5707963

File: urdf/urdf/robot_model.urdf (robot description, URDF)
Before this commit: robot Staubli, 7 links, 6 joints
Joints:
- joint Joint_1: origin xyz=0 0 0.375 rpy=-1.57 0 0 -> xyz=0 0 0.375 rpy=-1.5707963 0 0
- joint Joint_4: origin xyz=0 0 0 rpy=1.57 0 0 -> xyz=0 0 0 rpy=1.5707963 0 0
- joint Joint_5: origin xyz=0 0 0.45 rpy=-1.57 0 0 -> xyz=0 0 0.45 rpy=-1.5707963 0 0
- joint Joint_6: origin xyz=0 -0.07 0 rpy=1.57 0 0 -> xyz=0 -0.07 0 rpy=1.5707963 0 0

Commit message: ground

File: urdf/urdf/robot_model.urdf (robot description, URDF)
Before this commit: robot Staubli, 7 links, 6 joints
Links:
- added link Ground
Joints:
- added joint BaseJoint: type fixed, parent Ground, child base_link, origin xyz=0 0 0 rpy=0 0 0, axis 0 1 0, limit lower=-2.96 upper=2.96 effort=300 velocity=1
- joint Joint_1: origin xyz=0 0 0.375 rpy=-1.5707963 0 0 -> xyz=0 0 0 rpy=-1.5707963 0 0

Commit message: CalibrationAdaptor

File: urdf/urdf/robot_model.urdf (robot description, URDF)
Before this commit: robot Staubli, 8 links, 7 joints
Links:
- removed link Ground
- link base_link: geometry collision mesh filename=urdf/model/1.STL; visual mesh filename=urdf/model/1.STL
- link link_1: geometry collision mesh filename=urdf/model/2.STL; visual mesh filename=urdf/model/2.STL
- link link_2: geometry collision mesh filename=urdf/model\3.STL; visual mesh filename=urdf/model\3.STL
- link link_3: geometry collision mesh filename=urdf/model/4.STL; visual mesh filename=urdf/model\4.STL
- link link_4: geometry collision mesh filename=urdf/model/5.STL; visual mesh filename=urdf/model\5.STL
- link link_5: geometry collision mesh filename=urdf/model/6.STL; visual mesh filename=urdf/model/6.STL
- link link_6: geometry collision mesh filename=urdf/model/7.STL; visual mesh filename=urdf/model/7.STL
Joints:
- removed joint BaseJoint
- joint Joint_1: axis 0 1 0 -> 0 0 1; origin xyz=0 0 0 rpy=-1.5707963 0 0 -> xyz=0 0 0 rpy=0 0 0
- joint Joint_2: origin xyz=0.0 0.0 0.0 rpy=0 0 0 -> xyz=0.0 0.0 0.0 rpy=-1.5707963 0 0
